File: z90d_hardware.kicad_sch (KiCad schematic)
At the start: 3 parts, among them U1 ESP32-S3-WROOM-1, U2 ME6211C33M5, U3 PCM5102A

Commit message: alim
Parts:
- added C1: 10uF/25V, symbol Device:C
- added C2, C3: C, symbol Device:C
- added D1, D2, D3: LRC LESD5D5.0CT1G, Diode_SMD:D_SOD-523, symbol Device:D_TVS
- added D4: 1N5819HW-7-F, symbol Device:D
- added J1: USB_C_Receptacle_USB2.0_14P, Connector_USB:USB_C_Receptacle_GCT_USB4105-xx-A_16P_TopMnt_Horizontal, symbol Connector:USB_C_Receptacle_USB2.0_14P
- added J3: DE_15 Amplifier, symbol Connector:DE15_Socket_HighDensity
- added J4: DE15 Console, symbol Connector:DE15_Pins_HighDensity_MountingHoles
- added R1, R2: 5.1, symbol Device:R
- added U4: (no value), symbol lib:SGM2212
Connections:
- net GND: now reaches U1.1 (GND), U1.40 (GND), U1.41 (GND)
- net GND: now also C1.2, C2.2, C3.2, D1.1 (A1), D2.1 (A1), D3.1 (A1), J1.A1 (GND), J1.A12 (GND), J1.B1 (GND), J1.B12 (GND), J3.6, J4.6, J4.SH, R1.2, R2.2, U4.1 (GND)
- net GPIO19: now reaches U1.14 (USB_D+)
- net GPIO19: now also D2.2 (A2), J1.A7 (D-), J1.B7 (D-)
- net GPIO20: now reaches U1.23 (IO21)
- net GPIO20: now also D3.2 (A2), J1.A6 (D+), J1.B6 (D+)
- new net: J1.A5 (CC1), R2.1
- new net: J1.B5 (CC2), R1.1
- new net: D1.2 (A2), D4.2 (A), J1.A4 (VBUS), J1.A9 (VBUS), J1.B4 (VBUS), J1.B9 (VBUS)
- new net +5V: C1.1, C2.1, C3.1, D4.1 (K), U4.3 (VIN)
- new net audio_ground: J3.3, J4.3
- new net aux_left: J3.5
- new net aux_right: J3.4
- new net headphones_left: J3.2, J4.2
- new net headphones_right: J3.1, J4.1
- no-connect marks 0 -> 2
Other:
- moved on the sheet: U1, U2, U3
