File: z906_hardware.kicad_pcb (KiCad board)
At the start: 2 copper layers, 11 parts, among them J1 USB_C_Receptacle_USB2.0_14P, U1 ESP32-S3-WROOM-1, U2 AP63203WU, U3 PCM5102A, U4 TPD2EUSB30, U5 TPD1E05U06DYA, U6 TPS7A4533, U7 PCM1860DBT, U8 TPD2E2U06DCK

Commit message: pcb by claude
Parts:
- removed U8: TPD2E2U06DCK, Package_TO_SOT_SMD:SOT-323_SC-70
- added C1: 10uF, Capacitor_SMD:C_0805_2012Metric, F.Cu at (18.5, 18.7)
- added C10: 22uF, Capacitor_SMD:C_0805_2012Metric, F.Cu at (85.5, 21.0)
- added C11: 1uF, Capacitor_SMD:C_0603_1608Metric, F.Cu at (83.5, 27.0)
- added C14: 10uF, Capacitor_SMD:C_0805_2012Metric, F.Cu at (52.2, 14.2)
- added C15: 0.1uF, Capacitor_SMD:C_0603_1608Metric, F.Cu at (55.5, 14.2)
- added C16: 10uF, Capacitor_SMD:C_0805_2012Metric, F.Cu at (64.2, 14.2)
- added C17: 0.1uF, Capacitor_SMD:C_0603_1608Metric, F.Cu at (60.5, 14.2)
- added C18: 10uF, Capacitor_SMD:C_0805_2012Metric, F.Cu at (59.0, 25.5)
- added C19: 0.1uF, Capacitor_SMD:C_0603_1608Metric, F.Cu at (55.0, 25.5)
- added C2: 10uF, Capacitor_SMD:C_0805_2012Metric, F.Cu at (13.5, 43.5)
- added C20: 0.1uF, Capacitor_SMD:C_0603_1608Metric, F.Cu at (65.5, 17.0)
- added C21: 10uF, Capacitor_SMD:C_0805_2012Metric, F.Cu at (65.5, 19.2)
- added C22: 2.2uF, Capacitor_SMD:C_0603_1608Metric, F.Cu at (52.3, 18.4)
- added C23: 2.2uF, Capacitor_SMD:C_0603_1608Metric, F.Cu at (52.3, 24.5)
- added C24: 2.2nF, Capacitor_SMD:C_0603_1608Metric, F.Cu at (45.0, 17.0)
- added C25: 2.2nF, Capacitor_SMD:C_0603_1608Metric, F.Cu at (45.0, 21.0)
- added C26: 10uF, Capacitor_SMD:C_0805_2012Metric, F.Cu at (45.0, 36.5)
- added C27: 0.1uF, Capacitor_SMD:C_0603_1608Metric, F.Cu at (42.5, 36.5)
- added C28: 10uF, Capacitor_SMD:C_0805_2012Metric, F.Cu at (40.0, 36.5)
- added C29: 0.1uF, Capacitor_SMD:C_0603_1608Metric, F.Cu at (37.5, 36.5)
- added C30: 10uF, Capacitor_SMD:C_0805_2012Metric, F.Cu at (29.0, 31.5)
- added C31: 0.1uF, Capacitor_SMD:C_0603_1608Metric, F.Cu at (32.5, 31.5)
- added C32: 10uF, Capacitor_SMD:C_0805_2012Metric, F.Cu at (29.0, 33.6)
- added C33: 0.1uF, Capacitor_SMD:C_0603_1608Metric, F.Cu at (32.5, 33.2)
- added C34: 2.2uF, Capacitor_SMD:C_0603_1608Metric, F.Cu at (32.5, 29.8)
- added C35: 4.7uF, Capacitor_SMD:C_0603_1608Metric, F.Cu at (24.0, 22.0)
- added C36: 1nF, Capacitor_SMD:C_0603_1608Metric, F.Cu at (32.5, 26.4)
- added C37: 4.7uF, Capacitor_SMD:C_0603_1608Metric, F.Cu at (28.0, 22.0)
- added C38: 1nF, Capacitor_SMD:C_0603_1608Metric, F.Cu at (32.5, 28.1)
- added C4: 22uF, Capacitor_SMD:C_0805_2012Metric, F.Cu at (20.5, 48.5)
- added C6: 10uF, Capacitor_SMD:C_0805_2012Metric, F.Cu at (22.5, 57.0)
- added C7: 10uF, Capacitor_SMD:C_0805_2012Metric, F.Cu at (25.5, 53.0)
- added C8: 0.1uF, Capacitor_SMD:C_0603_1608Metric, F.Cu at (22.5, 53.0)
- added C9: 0.1uF, Capacitor_SMD:C_0603_1608Metric, F.Cu at (85.8, 23.5)
- added F1: 0ZLM0075FF2G, Fuse:Fuse_0603_1608Metric, F.Cu at (10.5, 18.6)
- added H1: M3, MountingHole:MountingHole_3.2mm_M3, F.Cu at (3.50, 3.50)
- added H2: M3, MountingHole:MountingHole_3.2mm_M3, F.Cu at (86.5, 3.50)
- added H3: M3, MountingHole:MountingHole_3.2mm_M3, F.Cu at (3.50, 56.5)
- added H4: M3, MountingHole:MountingHole_3.2mm_M3, F.Cu at (86.5, 56.5)
- added J3: DE_15 Amplifier, TerminalBlock:TerminalBlock_Xinya_XY308-2.54-15P_1x15_P2.54mm_Horizontal, F.Cu at (45.0, 4.20)
- added J4: DE15 Console, Connector_Dsub:DSUB-15-HD_Socket_Horizontal_P2.29x1.90mm_EdgePinOffset3.03mm_Housed_MountingHolesOffset4.94mm, F.Cu at (19.4, 6.83)
- added L1: 1.0uH, Inductor_SMD:L_Murata_DFE201610P, F.Cu at (17.0, 47.5)
- added R1: 5.1k, Resistor_SMD:R_0603_1608Metric, F.Cu at (12.0, 28.0)
- added R10: 100k, Resistor_SMD:R_0603_1608Metric, F.Cu at (24.0, 19.0)
- added R11: 100k, Resistor_SMD:R_0603_1608Metric, F.Cu at (28.0, 19.0)
- added R12: 100, Resistor_SMD:R_0603_1608Metric, F.Cu at (28.0, 25.0)
- added R2: 5.1k, Resistor_SMD:R_0603_1608Metric, F.Cu at (12.0, 21.0)
- added R3: 453k, Resistor_SMD:R_0603_1608Metric, F.Cu at (21.8, 43.0)
- added R4: 0, Resistor_SMD:R_0603_1608Metric, F.Cu at (88.0, 27.0)
- added R5: 10K, Resistor_SMD:R_0603_1608Metric, F.Cu at (85.8, 27.0)
- added R6: 470, Resistor_SMD:R_0603_1608Metric, F.Cu at (49.0, 20.3)
- added R7: 470, Resistor_SMD:R_0603_1608Metric, F.Cu at (49.0, 22.3)
- added R8: 100k, Resistor_SMD:R_0603_1608Metric, F.Cu at (21.8, 41.3)
- added R9: 100, Resistor_SMD:R_0603_1608Metric, F.Cu at (24.0, 25.0)
- added TP1: GND, Connector_Pin:Pin_D1.0mm_L10.0mm, F.Cu at (72.5, 53.0)
- added TP2: RXD0, Connector_Pin:Pin_D1.0mm_L10.0mm, F.Cu at (76.0, 53.0)
- added TP3: TXD0, Connector_Pin:Pin_D1.0mm_L10.0mm, F.Cu at (79.5, 53.0)
- added TP4: 3.3V, Connector_Pin:Pin_D1.0mm_L10.0mm, F.Cu at (88.3, 17.5)
- U2: value AP63203WU -> TPS62A02APDDC; footprint Package_TO_SOT_SMD:TSOT-23-6 -> Package_TO_SOT_SMD:SOT-23-6
- U6: footprint Package_TO_SOT_SMD:TO-263-5_TabPin3 -> Package_TO_SOT_SMD:SOT-223-6_TabPin3
- moved U7 165.8 mm to (40.0, 30.0)
- moved U3 143.7 mm to (58.0, 20.0)
- moved U5 141.6 mm to (15.5, 18.6), turned to -90 degrees
- moved U4 137.0 mm to (13.0, 24.0), turned to 90 degrees
- moved J1 134.6 mm to (3.60, 24.0)
- moved U2 125.3 mm to (18.0, 44.0)
- moved U6 118.5 mm to (16.0, 55.0), turned to 180 degrees
- moved U1 113.5 mm to (83.2, 40.0), turned to -90 degrees
- moved JP1 108.4 mm to (73.0, 21.0), turned to 0 degrees
- moved JP2 105.4 mm to (66.0, 53.0), turned to 0 degrees
Connections:
- J1 pad A4: +5V -> Net-(F1-Pad1)
- J1 pad A9: +5V -> Net-(F1-Pad1)
- J1 pad B4: +5V -> Net-(F1-Pad1)
- J1 pad B9: +5V -> Net-(F1-Pad1)
- U1 pad 36: unconnected-(U1-RXD0-Pad36) -> Net-(U1-RXD0)
- U1 pad 37: unconnected-(U1-TXD0-Pad37) -> Net-(U1-TXD0)
- U2 pad 1: +3.3V -> +5V
- U2 pad 2: +5V -> GND
- U2 pad 3: +5V -> Net-(U2-SW)
- U2 pad 4: GND -> +5V
- U2 pad 5: Net-(U2-SW) -> unconnected-(U2-PG-Pad5)
- U6 pad 1: Net-(U6-IN) -> +5V
- U6 pad 2: Net-(U6-IN) -> +5V
- U7 pad 19: Net-(U7-INT) -> unconnected-(U7-INT-Pad19)
Routing:
- net +3.3VA: track 0.00 -> 115.4 mm, vias 0 -> 9
- net /console_presence: track 0.00 -> 108.1 mm, vias 0 -> 3
- net /amplifier_presence: track 0.00 -> 85.2 mm, vias 0 -> 1
- net /USB_DN: track 0.00 -> 79.8 mm, vias 0 -> 4
- net /rx_console: track 0.00 -> 77.4 mm, vias 0 -> 4
- net /console_powered: track 0.00 -> 77.3 mm, vias 0 -> 1
- net /USB_DP: track 0.00 -> 76.8 mm, vias 0 -> 2
- net +5V: track 0.00 -> 71.2 mm
- net /tx_console: track 0.00 -> 68.7 mm, vias 0 -> 3
- net /MCLK: track 0.00 -> 60.0 mm
- net /BCK: track 0.00 -> 60.0 mm, vias 0 -> 2
- net /ADC_DATA: track 0.00 -> 59.5 mm, vias 0 -> 4
- net GND: track 0.00 -> 59.3 mm, vias 0 -> 112
- net /LCK: track 0.00 -> 55.4 mm, vias 0 -> 4
- net /logi_specific_2: track 0.00 -> 54.3 mm
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- added copper zone on In2.Cu, net +3.3V
- added copper zone on B.Cu, net GND
- added copper zone on F.Cu, net GND
- added copper zone on In1.Cu, net GND
Other:
- board outline added: 90 x 60 mm
- copper layers 2 -> 4
- board text added: "z906 ESP32-S3 audio bridge rev A"
